Commit message: Fix urdf in real world files

File: configs/urdf/realworld/sensors/d435i.urdf.xacro (robot description, xacro)
@@ -21,11 +21,8 @@
 <robot name="realsense2_camera" xmlns:xacro="http://www.ros.org/wiki/xacro">
   <xacro:arg name="name" default="camera" />
-  <xacro:arg name="topics_ns" default="realsense" />
   <xacro:arg name="use_nominal_extrinsics" default="true" />
-  <xacro:arg name="publish_pointcloud" default="false" />
-  <xacro:arg name="add_plug" default="false" />
   <xacro:include filename="$(find closedloop_nav_slam)/configs/urdf/turtlebot_properties_d435i.urdf.xacro"/>
   <xacro:include filename="$(find realsense2_description)/urdf/_d435i.urdf.xacro"/>
-  <xacro:sensor_d435i name="$(arg name)" topics_ns="$(arg topics_ns)" parent="base_link" use_nominal_extrinsics="$(arg use_nominal_extrinsics)" publish_pointcloud="$(arg publish_pointcloud)" add_plug="$(arg add_plug)">
+  <xacro:sensor_d435i name="$(arg name)" parent="base_link" use_nominal_extrinsics="$(arg use_nominal_extrinsics)">
     <origin xyz="${cam_px} ${cam_py} ${cam_pz}" rpy="${cam_or} ${cam_op} ${cam_oy}"/>
   </xacro:sensor_d435i>

File: configs/urdf/realworld/sensors/laser.urdf.xacro (robot description, xacro)
@@ -1,14 +1,14 @@
 <?xml version="1.0"?>
-<robot name="sensor_hokuyo" xmlns:xacro="http://ros.org/wiki/xacro">
+<robot name="sensor_laser" xmlns:xacro="http://ros.org/wiki/xacro">
   <xacro:include filename="$(find closedloop_nav_slam)/configs/urdf/turtlebot_properties_laser.urdf.xacro"/>
   <!-- Parameterised in part by the values in turtlebot_properties.urdf.xacro -->
-  <xacro:macro name="sensor_hokuyo" params="parent">
-    <joint name="hokuyo_joint" type="fixed">
+  <xacro:macro name="sensor_laser" params="parent">
+    <joint name="laser_joint" type="fixed">
       <axis xyz="0 1 0" />
-      <origin xyz="${lidar_px} ${lidar_py} ${lidar_pz}" rpy="${lidar_or} ${lidar_op} ${lidar_oy}"/>
+      <origin xyz="${laser_px} ${laser_py} ${laser_pz}" rpy="${laser_or} ${laser_op} ${laser_oy}"/>
       <parent link="${parent}"/>
       <child link="laser_link"/>
     </joint>
-    <!-- Hokuyo Laser -->
+    <!-- 2D Laser -->
     <link name="laser_link">
       <collision>
