Commit message: Change laser_link to laser frame

File: configs/urdf/gazebo/sensors/laser.urdf.xacro (robot description, xacro)
@@ -9,8 +9,8 @@
       <origin xyz="${laser_px} ${laser_py} ${laser_pz}" rpy="${laser_or} ${laser_op} ${laser_oy}"/>
       <parent link="${parent}"/>
-      <child link="laser_link"/>
+      <child link="laser"/>
     </joint>
     <!-- 2D Laser -->
-    <link name="laser_link">
+    <link name="laser">
       <collision>
         <origin xyz="0 0 0" rpy="0 0 0"/>

File: configs/urdf/gazebo/sensors/laser_sim.urdf.xacro (robot description, xacro)
@@ -3,5 +3,5 @@
   <xacro:macro name="turtlebot_sim_laser_sensor">
     <!-- hokuyo -->
-    <gazebo reference="laser_link">
+    <gazebo reference="laser">
       <sensor type="ray" name="head_laser_sensor">
         <always_on>true</always_on>
@@ -35,5 +35,5 @@
         <plugin name="gazebo_ros_head_laser_controller" filename="libgazebo_ros_laser.so">
           <topicName>/scan</topicName>
-          <frameName>laser_link</frameName>
+          <frameName>laser</frameName>
         </plugin>
       </sensor>

File: configs/urdf/realworld/sensors/laser.urdf.xacro (robot description, xacro)
@@ -8,8 +8,8 @@
       <origin xyz="${laser_px} ${laser_py} ${laser_pz}" rpy="${laser_or} ${laser_op} ${laser_oy}"/>
       <parent link="${parent}"/>
-      <child link="laser_link"/>
+      <child link="laser"/>
     </joint>
     <!-- 2D Laser -->
-    <link name="laser_link">
+    <link name="laser">
       <collision>
         <origin xyz="0 0 0" rpy="0 0 0"/>
