Commit message: Set sensor extrinsics

File: configs/urdf/turtlebot_properties_d435i.urdf.xacro (robot description, xacro)
@@ -7,9 +7,15 @@
     http://www.ros.org/reps/rep-0119.html
    -->
-	<xacro:property name="cam_px" value="0.15" />
+	<!-- <xacro:property name="cam_px" value="0.15" />
 	<xacro:property name="cam_py" value="0.0" />
 	<xacro:property name="cam_pz" value="0.3" />
 	<xacro:property name="cam_or" value="0" />
 	<xacro:property name="cam_op" value="0" />
+	<xacro:property name="cam_oy" value="0" /> -->
+ 	<xacro:property name="cam_px" value="0.114" />
+	<xacro:property name="cam_py" value="0.007" />
+	<xacro:property name="cam_pz" value="0.488" />
+	<xacro:property name="cam_or" value="0" />
+	<xacro:property name="cam_op" value="0" />
 	<xacro:property name="cam_oy" value="0" />
 </robot>

File: configs/urdf/turtlebot_properties_laser.urdf.xacro (robot description, xacro)
@@ -7,9 +7,15 @@
     http://www.ros.org/reps/rep-0119.html
    -->
-	<xacro:property name="laser_px" value="0.071" />
+	<!-- <xacro:property name="laser_px" value="0.071" />
 	<xacro:property name="laser_py" value="0.0" />
 	<xacro:property name="laser_pz" value="0.4" />
 	<xacro:property name="laser_or" value="0" />
 	<xacro:property name="laser_op" value="0" />
+	<xacro:property name="laser_oy" value="0" /> -->
+ 	<xacro:property name="laser_px" value="0.04" />
+	<xacro:property name="laser_py" value="0.0" />
+	<xacro:property name="laser_pz" value="0.35" />
+	<xacro:property name="laser_or" value="0" />
+	<xacro:property name="laser_op" value="0" />
 	<xacro:property name="laser_oy" value="0" />
 </robot>
