Commit message: Add 3D lidar SLAM
- hdl_slam, fast-lio2, liorf(lio-sam)
- Test in gazebo simulation

File: configs/urdf/gazebo/kobuki_hexagons_fisheye_stereo_mpu_6000_vlp16.urdf.xacro (robot description, xacro)
@@ -12,7 +12,9 @@
   <xacro:include filename="$(find closedloop_nav_slam)/configs/urdf/gazebo/sensors/fisheye_stereo.urdf.xacro"/>
   <xacro:include filename="$(find closedloop_nav_slam)/configs/urdf/gazebo/sensors/vlp16.urdf.xacro"/>
+  <xacro:include filename="$(find closedloop_nav_slam)/configs/urdf/gazebo/sensors/laser.urdf.xacro"/>
   <xacro:kobuki/>
   <xacro:stack_hexagons parent="base_link"/>
   <xacro:sensor_stereo  parent="base_link"/>
   <xacro:sensor_vlp16   parent="base_link" name="velodyne" topic="/velodyne_points" hz="10" samples="440" gpu="true"/>
+  <xacro:sensor_laser   parent="base_link"/>
 </robot>

File: configs/urdf/turtlebot_properties_laser.urdf.xacro (robot description, xacro)
@@ -15,5 +15,5 @@
  	<xacro:property name="laser_px" value="0.04" />
 	<xacro:property name="laser_py" value="0.0" />
-	<xacro:property name="laser_pz" value="0.35" />
+	<xacro:property name="laser_pz" value="0.4" />
 	<xacro:property name="laser_or" value="0" />
 	<xacro:property name="laser_op" value="0" />
